File: Documentation/Document Resources/XMICRO Backplane Dimenisons.brd (EAGLE design)
At the start: 203.2 x 70.6 mm, 5 parts

Commit message: Fixed dimensional drawings and pinout diagram
Changed lines of the file:
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@@
 <board>
 <plain>
-<wire x1="203.2" y1="52.705" x2="203.2" y2="109.22" width="0" layer="20"/>
-<wire x1="205.74" y1="109.22" x2="205.74" y2="52.705" width="0" layer="51" style="longdash"/>
+<wire x1="203.2" y1="52.705" x2="203.2" y2="109.22" width="0.0254" layer="20"/>
+<wire x1="205.74" y1="109.22" x2="205.74" y2="52.705" width="0.0254" layer="51" style="longdash"/>
 <text x="1.27" y="18.415" size="1.778" layer="51" font="vector" align="top-left">Notes:
 1. All dimensions are in inches.
@@
 5. All backplane slots must fit full-dimension cards.
 6. Maximum component height under cards may not exceed the edge connectors.</text>
-<wire x1="205.74" y1="63.5" x2="201.295" y2="67.945" width="0.0635" layer="48"/>
-<wire x1="201.295" y1="67.945" x2="194.31" y2="67.945" width="0.0635" layer="48"/>
-<wire x1="203.2" y1="85.09" x2="201.295" y2="86.995" width="0.0635" layer="48"/>
-<wire x1="201.295" y1="86.995" x2="193.04" y2="86.995" width="0.0635" layer="48"/>
+<wire x1="205.74" y1="63.5" x2="201.295" y2="67.945" width="0.0254" layer="48"/>
+<wire x1="201.295" y1="67.945" x2="194.31" y2="67.945" width="0.0254" layer="48"/>
+<wire x1="203.2" y1="85.09" x2="201.295" y2="86.995" width="0.0254" layer="48"/>
+<wire x1="201.295" y1="86.995" x2="193.04" y2="86.995" width="0.0254" layer="48"/>
 <text x="192.405" y="67.945" size="2.1844" layer="51" font="vector" rot="R180" align="center-left">INSIDE SURFACE OF CHASSIS</text>
 <text x="191.135" y="86.995" size="2.1844" layer="51" font="vector" rot="R180" align="center-left">BACKPLANE REAR PCB EDGE</text>
-<wire x1="152.4" y1="108.585" x2="152.4" y2="106.045" width="0.0635" layer="51"/>
-<wire x1="152.4" y1="106.045" x2="152.4" y2="103.505" width="0.0635" layer="51"/>
-<wire x1="152.4" y1="106.045" x2="205.74" y2="106.045" width="0.0635" layer="51"/>
-<polygon width="0.0635" layer="51">
+<wire x1="152.4" y1="108.585" x2="152.4" y2="106.045" width="0.0254" layer="51"/>
+<wire x1="152.4" y1="106.045" x2="152.4" y2="103.505" width="0.0254" layer="51"/>
+<wire x1="152.4" y1="106.045" x2="205.74" y2="106.045" width="0.0254" layer="51"/>
+<polygon width="0.0254" layer="51">
 <vertex x="203.2" y="106.045"/>
 <vertex x="202.08875" y="106.52125"/>
 <vertex x="202.08875" y="105.56875"/>
 </polygon>
-<polygon width="0.0635" layer="51">
+<polygon width="0.0254" layer="51">
 <vertex x="152.4" y="106.045"/>
 <vertex x="153.51125" y="105.56875"/>
@@
 </polygon>
 <text x="177.8" y="107.315" size="2.1844" layer="51" font="vector" align="bottom-center">2" TO CONNECTOR CENTER</text>
-<polygon width="0.254" layer="51">
+<polygon width="0.0254" layer="51">
 <vertex x="112.395" y="88.9"/>
 <vertex x="113.665" y="91.44"/>
@@
 </polygon>
 <text x="116.205" y="90.17" size="2.1844" layer="51" font="vector" align="center-left">PIN 1</text>
-<polygon width="0.254" layer="51">
+<polygon width="0.0254" layer="51">
 <vertex x="112.395" y="69.85"/>
 <vertex x="113.665" y="72.39"/>
 <vertex x="114.935" y="69.85"/>
 </polygon>
-<polygon width="0.254" layer="51">
+<polygon width="0.0254" layer="51">
 <vertex x="112.395" y="50.8"/>
 <vertex x="113.665" y="53.34"/>
 <vertex x="114.935" y="50.8"/>
 </polygon>
-<polygon width="0.254" layer="51">
+<polygon width="0.0254" layer="51">
 <vertex x="112.395" y="31.75"/>
 <vertex x="113.665" y="34.29"/>
 <vertex x="114.935" y="31.75"/>
 </polygon>
-<polygon width="0.0635" layer="51">
+<polygon width="0.0254" layer="51">
 <vertex x="205.74" y="63.5"/>
 <vertex x="205.26375" y="64.61125"/>
 <vertex x="204.62875" y="63.97625"/>
 </polygon>
-<polygon width="0.0635" layer="51">
+<polygon width="0.0254" layer="51">
 <vertex x="203.2" y="85.09"/>
 <vertex x="202.72375" y="86.20125"/>
 <vertex x="202.08875" y="85.56625"/>
 </polygon>
-<wire x1="103.505" y1="96.52" x2="106.045" y2="96.52" width="0.0635" layer="51"/>
-<wire x1="106.045" y1="96.52" x2="108.585" y2="96.52" width="0.0635" layer="51"/>
-<wire x1="103.505" y1="77.47" x2="106.045" y2="77.47" width="0.0635" layer="51"/>
-<wire x1="106.045" y1="77.47" x2="108.585" y2="77.47" width="0.0635" layer="51"/>
-<wire x1="106.045" y1="77.47" x2="106.045" y2="96.52" width="0.0635" layer="51"/>
+<wire x1="103.505" y1="96.52" x2="106.045" y2="96.52" width="0.0254" layer="51"/>
+<wire x1="106.045" y1="96.52" x2="108.585" y2="96.52" width="0.0254" layer="51"/>
+<wire x1="103.505" y1="77.47" x2="106.045" y2="77.47" width="0.0254" layer="51"/>
+<wire x1="106.045" y1="77.47" x2="108.585" y2="77.47" width="0.0254" layer="51"/>
+<wire x1="106.045" y1="77.47" x2="106.045" y2="96.52" width="0.0254" layer="51"/>
 <text x="103.505" y="86.995" size="2.1844" layer="51" font="vector" rot="R90" align="bottom-center">0.75"</text>
-<polygon width="0.0635" layer="51">
+<polygon width="0.0254" layer="51">
 <vertex x="106.045" y="96.52"/>
 <vertex x="105.56875" y="95.40875"/>
 <vertex x="106.52125" y="95.40875"/>
 </polygon>
-<polygon width="0.0635" layer="51">
+<polygon width="0.0254" layer="51">
 <vertex x="106.045" y="77.47"/>
 <vertex x="106.52125" y="78.58125"/>
@@
 </polygon>
 <rectangle x1="0" y1="38.57625" x2="203.2" y2="40.16375" layer="20"/>
-<wire x1="205.74" y1="42.70375" x2="205.74" y2="23.65375" width="0" layer="48" style="shortdash"/>
-<wire x1="205.74" y1="23.65375" x2="1.27" y2="23.65375" width="0" layer="48" style="shortdash"/>
-<wire x1="1.27" y1="23.65375" x2="1.27" y2="42.70375" width="0" layer="48" style="shortdash"/>
-<wire x1="1.27" y1="42.70375" x2="205.74" y2="42.70375" width="0" layer="48" style="shortdash"/>
+<wire x1="205.74" y1="42.70375" x2="205.74" y2="23.65375" width="0.0254" layer="48" style="shortdash"/>
+<wire x1="205.74" y1="23.65375" x2="1.27" y2="23.65375" width="0.0254" layer="48" style="shortdash"/>
+<wire x1="1.27" y1="23.65375" x2="1.27" y2="42.70375" width="0.0254" layer="48" style="shortdash"/>
+<wire x1="1.27" y1="42.70375" x2="205.74" y2="42.70375" width="0.0254" layer="48" style="shortdash"/>
 <text x="0.635" y="47.625" size="2.1844" layer="51" font="vector" align="center-left">CARD DIMENSIONS</text>
-<wire x1="43.18" y1="42.7101" x2="38.2651" y2="47.625" width="0.0635" layer="48"/>
-<wire x1="38.2651" y1="47.625" x2="30.48" y2="47.625" width="0.0635" layer="48"/>
-<polygon width="0.0635" layer="51">
+<wire x1="43.18" y1="42.7101" x2="38.2651" y2="47.625" width="0.0254" layer="48"/>
+<wire x1="38.2651" y1="47.625" x2="30.48" y2="47.625" width="0.0254" layer="48"/>
+<polygon width="0.0254" layer="51">
 <vertex x="43.18" y="42.7101"/>
 <vertex x="42.70375" y="43.82135"/>
 <vertex x="42.06875" y="43.18635"/>
 </polygon>
-<polygon width="0.0635" layer="51">
+<polygon width="0.0254" layer="51">
 <vertex x="205.74" y="106.045"/>
 <vertex x="204.94625" y="106.52125"/>
 <vertex x="204.94625" y="105.56875"/>
 </polygon>
-<polygon width="0.0635" layer="51">
+<polygon width="0.0254" layer="51">
 <vertex x="203.2" y="106.045"/>
 <vertex x="203.99375" y="105.56875"/>
 <vertex x="203.99375" y="106.52125"/>
 </polygon>
-<text x="204.47" y="111.125" size="2.1844" layer="51" font="vector" align="bottom-center">0.1"</text>
-<wire x1="115.8875" y1="101.2825" x2="111.125" y2="106.045" width="0.0635" layer="48"/>
-<wire x1="111.125" y1="106.045" x2="104.14" y2="106.045" width="0.0635" layer="48"/>
+<text x="208.28" y="107.315" size="2.1844" layer="51" font="vector">0.1"</text>
+<wire x1="115.8875" y1="101.2825" x2="111.125" y2="106.045" width="0.0254" layer="48"/>
+<wire x1="111.125" y1="106.045" x2="104.14" y2="106.045" width="0.0254" layer="48"/>
 <text x="102.235" y="106.045" size="2.1844" layer="51" font="vector" rot="R180" align="center-left">CARD SLOT 0</text>
-<polygon width="0.0635" layer="51">
+<polygon width="0.0254" layer="51">
 <vertex x="115.8875" y="101.2825"/>
 <vertex x="115.41125" y="102.39375"/>
@@
 </polygon>
 <text x="3.81" y="86.36" size="2.1844" layer="51" font="vector" align="center-left">SYSTEM FRONT</text>
-<polygon width="0.4064" layer="51">
+<polygon width="0.0254" layer="51">
 <vertex x="2.54" y="87.63"/>
 <vertex x="2.54" y="85.09"/>
 <vertex x="0" y="86.36"/>
 </polygon>
-<polygon width="0.254" layer="51">
+<polygon width="0.0254" layer="51">
 <vertex x="112.395" y="12.7"/>
 <vertex x="113.665" y="15.24"/>
