File: Tools/xmicro-breakout/Hardware/CAD/XMICRO-BREAKOUT-CARD.brd (EAGLE design)
At the start: 101.6 x 30.5 mm, 3 parts, among them J1 HDR-17X2, J2 HDR-17X2, P1 XMICRO-BUS-PHYSICAL-EDGE62M

Commit message: Fixed tools with new IOSEL signal
Connections:
- net CLKAUX renamed !IOSEL
Changed lines of the file:
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@@
 <wire x1="21.59" y1="31.75" x2="20.32" y2="33.02" width="0.254" layer="1"/>
 </signal>
-<signal name="CLKAUX">
+<signal name="!IOSEL">
 <contactref element="P1" pad="16"/>
 <wire x1="30.48" y1="4.6101" x2="30.48" y2="8.255" width="0.254" layer="16"/>
