File: Documentation/Document Resources/Physical Diagrams/XMICRO Card Dimensions.brd (EAGLE design)
At the start: 228.6 x 109.2 mm, 0 parts

Commit message: Updated timing specs, changed physical drawings font
Other:
- board text added: "0.1""
- board text added: "2""
- board text added: "CARD REAR PCB EDGE"
- board text added: "INSIDE SURFACE OF CHASSIS"
- board text added: "NOTES: 1. All dimensions are specified in inches 2. Omit center mounting holes on full-size cards"
- board text removed: "0.1" TO INSIDE SURFACE OF CHASSIS"
- board text removed: "2" TO CONNECTOR CENTER"
- board text removed: "FRONT"
- board text removed: "NOTES: 1. All dimensions are in inches 2. Omit center mounting holes on full-size cards"
- board text removed: "REAR"
