File: Documentation/Document Resources/Physical Diagrams/XMICRO Backplane Dimenisons.brd (EAGLE design)
At the start: 0 parts

Commit message: Minor documentation improvements
Other:
- board text removed: "NOTES: 1. All dimensions are specified in inches 2. Minimum chassis clearance 0.0" to rear edge"
Changed lines of the file:
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@@
 <plain>
 <wire x1="203.2" y1="41.275" x2="203.2" y2="94.615" width="0.1016" layer="51"/>
-<text x="1.27" y="5.715" size="1.778" layer="51" align="top-left">NOTES:
-1. All dimensions are specified in inches
-2. Minimum chassis clearance 0.0" to rear edge</text>
 <wire x1="203.2" y1="94.615" x2="203.2" y2="97.79" width="0.1016" layer="51"/>
 <wire x1="203.2" y1="71.12" x2="198.755" y2="75.565" width="0.1016" layer="51"/>
@@
 </board>
 </drawing>
-<compatibility>
-<note version="6.3" minversion="6.2.2" severity="warning">
-Since Version 6.2.2 text objects can contain more than one line,
-which will not be processed correctly with this version.
-</note>
-</compatibility>
 </eagle>
